File: gbcartext.kicad_pcb (KiCad board)
At the start: 2 copper layers, 56 x 82.7 mm, 13 parts

Commit message: Add files via upload
Made it better with the improvement of my ability :-)
Parts:
- added G***: LOGO, LOGO, F.Cu at (140.3, 64.8)
- moved REF** 1.27 mm to (188.6, 111.8)
- moved REF** 0.63 mm to (188.6, 80.0)
Connections:
- REF** pad 10: (no net) -> GND (x2)
- REF** pad 13: (no net) -> GND (x2)
- REF** pad 26: (no net) -> GND (x2)
- REF** pad 5: (no net) -> GND (x5)
- REF** pad 3: (no net) -> GND
- REF** pad 1: (no net) -> GND (x2)
- REF** pad 2: (no net) -> GND
- REF** pad 4: (no net) -> GND
Routing:
- net GND: track 0.00 -> 239.5 mm
- net (no net): track 852.4 -> 615.7 mm, vias 18 -> 17
- added copper zone on B.Cu, net GND
- added copper zone on F.Cu, net GND
Other:
- outline, holes or cut-outs redrawn
